Commit message: Add thumb

File: simulation_environment/models/hand/hand.xacro (robot description, xacro)
@@ -30,11 +30,14 @@
   </link>
   <!-- Add the fingers -->
-  <xacro:finger prefix="pinkie_finger" parent="base_link" length1="${pinkie_l1}"
-      length2="${pinkie_l2}" length3="${pinkie_l3}" radius="${pinkie_r}" density="${density}" base_xyz="${-x_base/2 + pinkie_r} ${y_base/2} 0"/>
-  <xacro:finger prefix="ring_finger" parent="base_link" length1="${ring_l1}"
-      length2="${ring_l2}" length3="${ring_l3}" radius="${ring_r}" density="${density}" base_xyz="${-x_base/2 + 2*pinkie_r + ring_r + 0.002} ${y_base/2} 0"/>
-  <xacro:finger prefix="middle_finger" parent="base_link" length1="${middle_l1}"
-      length2="${middle_l2}" length3="${middle_l3}" radius="${middle_r}" density="${density}" base_xyz="${-x_base/2 + 2*pinkie_r + 2*ring_r + middle_r + 0.003} ${y_base/2} 0"/>
-  <xacro:finger prefix="index_finger" parent="base_link" length1="${index_l1}"
-      length2="${index_l2}" length3="${index_l3}" radius="${index_r}" density="${density}" base_xyz="${x_base/2 - index_r} ${y_base/2} 0"/>
+  <xacro:finger prefix="pinkie_finger" parent="base_link" length1="${pinkie_l1}" length2="${pinkie_l2}" length3="${pinkie_l3}"
+      radius="${pinkie_r}" density="${density}" base_xyz="${-x_base/2 + pinkie_r} ${y_base/2} 0" base_rpy="${-pi/2} 0 0"/>
+  <xacro:finger prefix="ring_finger" parent="base_link" length1="${ring_l1}" length2="${ring_l2}" length3="${ring_l3}"
+      radius="${ring_r}" density="${density}" base_xyz="${-x_base/2 + 2*pinkie_r + ring_r + 0.002} ${y_base/2} 0" base_rpy="${-pi/2} 0 0"/>
+  <xacro:finger prefix="middle_finger" parent="base_link" length1="${middle_l1}" length2="${middle_l2}" length3="${middle_l3}"
+      radius="${middle_r}" density="${density}" base_xyz="${-x_base/2 + 2*pinkie_r + 2*ring_r + middle_r + 0.003} ${y_base/2} 0" base_rpy="${-pi/2} 0 0"/>
+  <xacro:finger prefix="index_finger" parent="base_link" length1="${index_l1}" length2="${index_l2}" length3="${index_l3}"
+      radius="${index_r}" density="${density}" base_xyz="${x_base/2 - index_r} ${y_base/2} 0" base_rpy="${-pi/2} 0 0"/>
+  <!-- Add the thumb -->
+  <xacro:finger prefix="thumb" parent="base_link" length1="${thumb_l1}" length2="${thumb_l2}" length3="${thumb_l3}"
+      radius="${thumb_r}" density="${density}" base_xyz="${x_base/2 - 0.707*thumb_r} ${-y_base/2 + 0.707*thumb_r} 0" base_rpy="${-pi/2} ${-pi/4} ${-pi/3}"/>
  </robot>

File: simulation_environment/models/hand/macros.xacro (robot description, xacro)
@@ -45,6 +45,6 @@
   </xacro:macro>
   <!-- Define the complete finger -->
-  <xacro:macro name="finger" params="prefix parent length1 length2 length3 radius density base_xyz">
-		<xacro:finger_part prefix="${prefix}" parent="${parent}" part="1" length="${length1}" radius="${radius}" density="${density}" origin_xyz="${base_xyz}" origin_rpy="${-pi/2} 0 0" />
+  <xacro:macro name="finger" params="prefix parent length1 length2 length3 radius density base_xyz base_rpy">
+		<xacro:finger_part prefix="${prefix}" parent="${parent}" part="1" length="${length1}" radius="${radius}" density="${density}" origin_xyz="${base_xyz}" origin_rpy="${base_rpy}" />
 		<xacro:finger_part prefix="${prefix}" parent="${prefix}_link_1" part="2" length="${length2}" radius="${radius}" density="${density}" origin_xyz="0 0 ${length1}" origin_rpy="0 0 0"/>
 		<xacro:finger_part prefix="${prefix}" parent="${prefix}_link_2" part="3" length="${length3}" radius="${radius}" density="${density}" origin_xyz="0 0 ${length2}" origin_rpy="0 0 0"/>

File: simulation_environment/models/hand/parameter.xacro (robot description, xacro)
@@ -31,6 +31,7 @@
   <xacro:property name="index_r" value="0.01125" />
   <!-- thumb -->
-  <xacro:property name="thumb_l1" value="0.0325" />
-  <xacro:property name="thumb_l2" value="0.03" />
-  <xacro:property name="ring_r" value="0.01375" />
+  <xacro:property name="thumb_l1" value="0.055" />
+  <xacro:property name="thumb_l2" value="0.0325" />
+  <xacro:property name="thumb_l3" value="0.03" />
+  <xacro:property name="thumb_r" value="0.01375" />
 </robot>
